File: rev_a/atum.sch (EAGLE design)
At the start: 41 parts, among them J1 EPIC2-HEADER2, J2 SH_MALE_2/1MM, U1 TPS62740, U2 FM25LBTDFN-8, U3 CC2538, U5 RV-3049-C3, X1 EPSON-FA-128, X3 ABS05-32.768KHZ-T

Commit message: updated silkscreen and names
- renumbered parts
- made silkscreen names for assembly
Parts:
- removed U5: RV-3049-C3, chips:RV-3049-C3
- added U4: TPS62740, chips:TPS62740
- C13, C14, C15: value 1uF -> 0.1uF
- C16, C17: value 22pF -> 1uF
- C18: value 10uF -> 1uF; device passives:CAPACITOR0603_CAP -> passives:CAPACITOR; DIGIKEY 490-7316-1-ND -> (none)
- C19: DIGIKEY 1276-1119-1-ND -> 490-7316-1-ND
- C20: value 0.1uF -> 10uF; device rcl:C-EUC0201 -> passives:CAPACITOR0603_CAP; DIGIKEY (none) -> 490-7316-1-ND
- C3: value 220pF -> 22pF
- C4: value 1nF -> 22pF
- C5: value 0.1uF -> 220pF
- C6: value 0.1uF -> 1nF
- C8: device passives:CAPACITOR -> rcl:C-EUC0201
- R1: value 2.2k -> 1k
- R4: value 1k -> 2.2k
- R6: value 56k -> 10k
- R7: value 10k -> 56k
- U1: value TPS62740 -> CC2538; device chips:TPS62740 -> chips:CC2538
- U3: value CC2538 -> RV-3049-C3; device chips:CC2538 -> chips:RV-3049-C3
- renumbered A2 to A1, X3 to X2
Connections:
- net !FRAM_CS: now also U1.PD1; no longer U3.PD1
- net !FRAM_HOLD: now also U1.PD0; no longer U3.PD0
- net !FRAM_WP: now also U1.PD2; no longer U3.PD2
- net !RESET: now also R4.1; no longer R1.1
- net !RTC_INT: now also U1.PB2, U3.!INT; no longer U3.PB2, U5.!INT
- net ADC3: now also U1.PA3/ROM-SSI-SEL; no longer U3.PA3/ROM-SSI-SEL
- net ADC4: now also U1.PA4/ROM-SSI-RX; no longer U3.PA4/ROM-SSI-RX
- net ADC5: now also U1.PA5/ROM-SSI-TX; no longer U3.PA5/ROM-SSI-TX
- net ADC6: now also U1.PA6; no longer U3.PA6
- net ADC7: now also U1.PA7; no longer U3.PA7
- net B3: now also U1.PB3; no longer U3.PB3
- net B4: now also U1.PB4; no longer U3.PB4
- net B5: now also U1.PB5; no longer U3.PB5
- net B6: now also U1.PB6/JTAG-TDI; no longer U3.PB6/JTAG-TDI
- net BATTERY: now also C19.1, U4.EN, U4.VIN, U4.VSEL2, U4.VSEL4; no longer C18.1, U1.EN, U1.VIN, U1.VSEL2, U1.VSEL4
- net BOOTLOADER_CTRL: now also U1.PA2/ROM-SSI-CLK; no longer U3.PA2/ROM-SSI-CLK
- net BOOTLOADER_RX: now also U1.PA0/ROM-UART-RX; no longer U3.PA0/ROM-UART-RX
- net BOOTLOADER_TX: now also U1.PA1/ROM-UART-TX; no longer U3.PA1/ROM-UART-TX
- net C0: now also U1.PC0; no longer U3.PC0
- net C1: now also U1.PC1; no longer U3.PC1
- net C2: now also U1.PC2; no longer U3.PC2
- net C3: now also U1.PC3; no longer U3.PC3
- net DGND_USB: now also U1.DGND_USB; no longer U3.DGND_USB
- net DVDD_USB: now also U1.DVDD_USB; no longer U3.DVDD_USB
- net GND: now also R6.1, R7.2, U4.CTRL, U4.GND, U4.VSEL1, U4.VSEL3; no longer R6.2, R7.1, U1.CTRL, U1.VSEL1, U1.VSEL3, U5.GND
- net I2C_SCL: now also U1.PC4; no longer U3.PC4
- net I2C_SDA: now also U1.PC5; no longer U3.PC5
- net LED_BLUE: now also R3.2, U1.PD4; no longer R4.2, U3.PD4
- net LED_GREEN: now also R2.2, U1.PD5; no longer R3.2, U3.PD5
- net LED_RED: now also R1.2, U1.PD3; no longer R2.2, U3.PD3
- net N$1: now also C6.1, R4.2, U1.!RESET; no longer C4.1, R1.2, U3.!RESET
- net N$10: now also U1.XOSC32M_Q2; no longer U3.XOSC32M_Q2
- net N$11: now also R2.1; no longer R3.1
- net N$12: now also R3.1; no longer R4.1
- net N$13: now also C4.1, U1.PD7/XOSC32K_Q2; no longer C17.1, U3.PD7/XOSC32K_Q2
- net N$14: now also R6.2, U3.VBACKUP; no longer R7.2, U5.VBACKUP
- net N$15: now also C17.1, C18.1, U1.DCOUPL1, U1.DCOUPL2; no longer C14.1, C15.1, U3.DCOUPL1, U3.DCOUPL2
- net N$16: now also U3.CLKOE; no longer U5.CLKOE
- net N$5: now also U4.SW; no longer U1.SW
- net N$6: now also C3.1, U1.PD6/XOSC32K_Q1; no longer C16.1, U3.PD6/XOSC32K_Q1
- net N$7: now also R1.1; no longer R2.1
- net N$8: now also R7.1, U1.R_BIAS; no longer R6.1, U3.R_BIAS
- net N$9: now also U1.XOSC32M_Q1; no longer U3.XOSC32M_Q1
- net RF_N: now also U1.RF_N; no longer U3.RF_N
- net RF_P: now also U1.RF_P; no longer U3.RF_P
- net RTC_CE: now also U1.PB1, U3.CE; no longer U3.PB1, U5.CE
- net SPI_MISO: now also U1.PB0, U3.MISO; no longer U3.PB0, U5.MISO
- net SPI_MOSI: now also U1.PC7, U3.MOSI; no longer U3.PC7, U5.MOSI
- net SPI_SCK: now also U1.PC6, U3.SCL; no longer U3.PC6, U5.SCL
- net TCK: now also U1.JTAG_TCK; no longer U3.JTAG_TCK
- net TDO: now also U1.PB7/JTAG-TDO; no longer U3.PB7/JTAG-TDO
- net TMS: now also U1.JTAG_TMS; no longer U3.JTAG_TMS
- net USB_N: now also U1.USB_N; no longer U3.USB_N
- net USB_P: now also U1.USB_P; no longer U3.USB_P
- net VCC: now also C14.1, C15.1, C16.1, U1.AVDD, U1.AVDD_GUARD, U1.DVDD, U3.VCC, U4.VOUT; no longer C19.1, C3.1, C6.1, U1.VOUT, U3.AVDD, U3.AVDD_GUARD, U3.DVDD, U5.VCC
Other:
- moved on the sheet: C10, C11, C12, C13, C14, C15, C16, C17, C19, C3, C4, C5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
