File: hardware/atum/rev_a/atum.brd (EAGLE design)
At the start: 18.8 x 19.6 mm, 41 parts, among them J1 EPIC2-HEADER2, J2 SH_MALE_2/1MM, U1 CC2538, U2 FM25LBTDFN-8, U3 RV-3049-C3, U4 TPS62740, X1 EPSON-FA-128, X2 ABS05-32.768KHZ-T

Commit message: trying to improve castellations
Parts:
- removed J1: EPIC2-HEADER2, epic2:EPIC2-HEADER2
- added J3: ATUM-HEADER, atum:ATUM-HEADER
- moved C9 0.36 mm to (9.07, 16.5)
- moved LOGO1 0.20 mm to (1.73, 8.56)
- moved C8 0.08 mm to (17.5, 8.59)
Connections:
- net !RESET: now also J3.30, J3.30B; no longer J1.30
- net ADC3: now also J3.25, J3.25B; no longer J1.25
- net ADC4: now also J3.26, J3.26B; no longer J1.26
- net ADC5: now also J3.27, J3.27B; no longer J1.27
- net ADC6: now also J3.28, J3.28B; no longer J1.28
- net ADC7: now also J3.29, J3.29B; no longer J1.29
- net B3: now also J3.9, J3.9B; no longer J1.9
- net B4: now also J3.8, J3.8B; no longer J1.8
- net B5: now also J3.7, J3.7B; no longer J1.7
- net B6: now also J3.6, J3.6B; no longer J1.6
- net BATTERY: now also J3.31, J3.31B; no longer J1.31
- net BOOTLOADER_CTRL: now also J3.24, J3.24B; no longer J1.24
- net BOOTLOADER_RX: now also J3.22, J3.22B; no longer J1.22
- net BOOTLOADER_TX: now also J3.23, J3.23B; no longer J1.23
- net C0: now also J3.21, J3.21B; no longer J1.21
- net C1: now also J3.20, J3.20B; no longer J1.20
- net C2: now also J3.19, J3.19B; no longer J1.19
- net DGND_USB: now also J3.10, J3.10B; no longer J1.10
- net DVDD_USB: now also J3.13, J3.13B; no longer J1.13
- net GND: now also J3.32, J3.32B; no longer J1.32
- net I2C_SCL: now also J3.17, J3.17B; no longer J1.17
- net I2C_SDA: now also J3.18, J3.18B; no longer J1.18
- net SPI_MISO: now also J3.14, J3.14B; no longer J1.14
- net SPI_MOSI: now also J3.15, J3.15B; no longer J1.15
- net SPI_SCK: now also J3.16, J3.16B; no longer J1.16
- net TCK: now also J3.4, J3.4B; no longer J1.4
- net TDO: now also J3.5, J3.5B; no longer J1.5
- net TMS: now also J3.3, J3.3B; no longer J1.3
- net UNUSED1: now also J3.2, J3.2B; no longer J1.2
- net USB_N: now also J3.12, J3.12B; no longer J1.12
- net USB_P: now also J3.11, J3.11B; no longer J1.11
- net VCC: now also J3.1, J3.1B; no longer J1.1
Routing:
- net VCC: track 39.4 -> 41.6 mm
