File: hardware/atum/rev_a/atum.brd (EAGLE design)
At the start: 18.8 x 19.6 mm, 41 parts, among them J2 SH_MALE_2/1MM, J3 ATUM-HEADER, U1 CC2538, U2 FM25LBTDFN-8, U3 RV-3049-C3, U4 TPS62740, X1 EPSON-FA-128, X2 ABS05-32.768KHZ-T

Commit message: new atum a
designed for advanced circuits default stack
Parts:
- moved C11 0.13 mm to (16.2, 12.0)
- moved C7 0.11 mm to (14.5, 17.2)
- moved C16 0.10 mm to (16.0, 1.85)
- moved C18 0.08 mm to (16.8, 1.85)
- moved R6 0.08 mm to (14.8, 13.3)
- moved C4 0.08 mm to (10.2, 1.24)
- moved R5 0.05 mm to (16.8, 15.3)
Routing:
- net I2C_SDA: track 6.58 -> 5.92 mm
Other:
- board text added: "2014/08/04"
- board text removed: "2014/04/28"
