File: hardware/atum/rev_a/atum.sch (EAGLE design)
At the start: 41 parts, among them J1 EPIC2-HEADER2, J2 SH_MALE_2/1MM, U1 CC2538, U2 FM25LBTDFN-8, U3 RV-3049-C3, U4 TPS62740, X1 EPSON-FA-128, X2 ABS05-32.768KHZ-T

Commit message: trying to improve castellations
Parts:
- removed J1: EPIC2-HEADER2, epic2:EPIC2-HEADER2
- added J3: ATUM-HEADER, atum:ATUM-HEADER
Connections:
- net !RESET: now also J3.30; no longer J1.30
- net ADC3: now also J3.25; no longer J1.25
- net ADC4: now also J3.26; no longer J1.26
- net ADC5: now also J3.27; no longer J1.27
- net ADC6: now also J3.28; no longer J1.28
- net ADC7: now also J3.29; no longer J1.29
- net B3: now also J3.9; no longer J1.9
- net B4: now also J3.8; no longer J1.8
- net B5: now also J3.7; no longer J1.7
- net B6: now also J3.6; no longer J1.6
- net BATTERY: now also J3.31; no longer J1.31
- net BOOTLOADER_CTRL: now also J3.24; no longer J1.24
- net BOOTLOADER_RX: now also J3.22; no longer J1.22
- net BOOTLOADER_TX: now also J3.23; no longer J1.23
- net C0: now also J3.21; no longer J1.21
- net C1: now also J3.20; no longer J1.20
- net C2: now also J3.19; no longer J1.19
- net DGND_USB: now also J3.10; no longer J1.10
- net DVDD_USB: now also J3.13; no longer J1.13
- net GND: now also J3.32; no longer J1.32
- net I2C_SCL: now also J3.17; no longer J1.17
- net I2C_SDA: now also J3.18; no longer J1.18
- net SPI_MISO: now also J3.14; no longer J1.14
- net SPI_MOSI: now also J3.15; no longer J1.15
- net SPI_SCK: now also J3.16; no longer J1.16
- net TCK: now also J3.4; no longer J1.4
- net TDO: now also J3.5; no longer J1.5
- net TMS: now also J3.3; no longer J1.3
- net UNUSED1: now also J3.2; no longer J1.2
- net USB_N: now also J3.12; no longer J1.12
- net USB_P: now also J3.11; no longer J1.11
- net VCC: now also J3.1; no longer J1.1
